Commit message: [Local Modification Backup] + something Jeong-woo knows :)

File: summit_xl_description/robots/summit_xl.urdf.xacro (robot description, xacro)
@@ -49,4 +49,7 @@
 			<origin xyz="0.19 0 0.26" rpy="0 ${15*PI/180} 0"/>
 		</xacro:sensor_axis-->
+		<!--xacro:sensor_vlp16 prefix="$(arg prefix)front_laser" parent="$(arg prefix)base_link" prefix_topic="front_laser">
+			<origin xyz="0.0 0.0 0.33" rpy="0 0 0"/>
+		</xacro:sensor_vlp16-->
 	    <!-- RGBD -->
 	    <!--xacro:sensor_orbbec_astra prefix="$(arg prefix)front_rgbd_camera" parent="$(arg prefix)base_link" prefix_topic="front_rgbd_camera">
