Commit message: + waterloo steel

File: summit_xl_description/robots/versions/summit_xls_171102A.urdf.xacro (robot description, xacro)
@@ -70,19 +70,10 @@
 			<origin xyz="${front_laser_offset_x} ${front_laser_offset_y} ${front_laser_offset_z}" rpy="0 0 0"/>
 		</xacro:sensor_vlp16>
-		<!--xacro:sensor_hokuyo_ust10lx prefix="$(arg prefix)front_laser" parent="$(arg prefix)base_link" prefix_topic="front_laser">
-			<origin xyz="${front_laser_offset_x} ${front_laser_offset_y} ${front_laser_offset_z}" rpy="0 0 ${-PI/4.0}"/>
-		</xacro:sensor_hokuyo_ust10lx-->
-		<!--xacro:sensor_hokuyo_ust10lx prefix="$(arg prefix)rear_laser" parent="$(arg prefix)base_link" prefix_topic="rear_laser">
-			<origin xyz="${rear_laser_offset_x} ${rear_laser_offset_y} ${rear_laser_offset_z}" rpy="0 0 ${3.0*PI/4.0}"/>
-		</xacro:sensor_hokuyo_ust10lx-->
 		<!-- <xacro:sensor_orbbec_astra prefix="$(arg prefix)front_rgbd_camera" parent="$(arg prefix)base_link" prefix_topic="front_rgbd_camera">
 			<origin xyz="${front_rgbd_camera_offset_x} ${front_rgbd_camera_offset_y} ${front_rgbd_camera_offset_z}" rpy="0 0 0"/>
 		</xacro:sensor_orbbec_astra> -->
-		<!--xacro:sensor_gps prefix="$(arg prefix)gps" parent="$(arg prefix)base_link">
-			<origin xyz="${gps_offset_x} ${gps_offset_y} ${gps_offset_z}" rpy="0 0 0"/>
-		</xacro:sensor_gps-->
-   </xacro:macro>
-   <!-- Gazebo ros control pluggins -->
-   <xacro:ros_control/>
-   <xacro:summit_xl prefix="$(arg prefix)" publish_bf="true" hq="true"/>
+	</xacro:macro>
+	<!-- Gazebo ros control pluggins -->
+	<xacro:ros_control/>
+	<xacro:summit_xl prefix="$(arg prefix)" publish_bf="true" hq="true"/>
 </robot>

Commit message: + added wheel radius attribute

File: summit_xl_description/robots/versions/summit_xls_171102A.urdf.xacro (robot description, xacro)
@@ -15,4 +15,5 @@
 	<xacro:property name="PI" value="3.1415926535897931"/>
 	<!-- Wheel parameters -->
+	<xacro:property name="wheel_radius" value="0.127" /> <!-- omin-wheel -->
 	<xacro:property name="wheel_offset_x" value="0.2225" />    <!-- x,y,z in translation from base_link to the center of the wheel -->
 	<xacro:property name="wheel_offset_y" value="0.2045" />
@@ -67,7 +68,7 @@
 		</xacro:structure_laser-->
 		<!-- SENSORS -->
-		<xacro:sensor_vlp16 prefix="$(arg prefix)front_laser" parent="$(arg prefix)base_link">
-			<origin xyz="${front_laser_offset_x} ${front_laser_offset_y} ${front_laser_offset_z}" rpy="0 0 0"/>
-		</xacro:sensor_vlp16>
+		<xacro:sensor_velodyne_vlp16 prefix="$(arg prefix)front_laser" parent="$(arg prefix)base_link" range_min="0.4" range_max="130">
+			<origin xyz="${front_laser_offset_x} ${front_laser_offset_y} ${front_laser_offset_z}" rpy="0 0 0" /> <!-- [m] -->
+		</xacro:sensor_velodyne_vlp16>
 		<!-- <xacro:sensor_orbbec_astra prefix="$(arg prefix)front_rgbd_camera" parent="$(arg prefix)base_link" prefix_topic="front_rgbd_camera">
 			<origin xyz="${front_rgbd_camera_offset_x} ${front_rgbd_camera_offset_y} ${front_rgbd_camera_offset_z}" rpy="0 0 0"/>
